File: ControlModule/CMBoard/CMBoard.kicad_pcb (KiCad board)
At the start: 2 copper layers, 22 x 80 mm, 2 parts, among them IC1 ESP32-S3-WROOM-1U-N4

Commit message: Initial commit
Parts:
- added C1: GRM219R60J476ME44D, SamacSys_Parts:GRM21BR60J226ME39L, F.Cu at (169.6, 84.9)
- added C2: 22u, Capacitor_SMD:C_0603_1608Metric, F.Cu at (169.9, 90.0)
- added C3: 22u, Capacitor_SMD:C_0603_1608Metric, F.Cu at (176.2, 71.6)
- added C4: GRM219R60J476ME44D, SamacSys_Parts:GRM21BR60J226ME39L, F.Cu at (176.1, 66.5)
- added C5: 10u, Capacitor_SMD:C_0603_1608Metric, B.Cu at (150.0, 82.1)
- added C6: 0u1, Capacitor_SMD:C_0603_1608Metric, B.Cu at (151.5, 82.1)
- added C7: 47n, Capacitor_SMD:C_0603_1608Metric, B.Cu at (148.4, 81.0)
- added C8: 4u7, Capacitor_SMD:C_0603_1608Metric, F.Cu at (147.0, 83.0)
- added C9: 20u, Capacitor_SMD:C_0603_1608Metric, F.Cu at (146.0, 87.1)
- added J1: GSB1C41110SSHR, SamacSys_Parts:GSB1C41110SSHR, F.Cu at (197.4, 97.1)
- added JP1: SolderJumper_3_Open, Jumper:SolderJumper-3_P1.3mm_Open_Pad1.0x1.5mm, B.Cu at (175.9, 88.4)
- added JP2: SolderJumper_3_Open, Jumper:SolderJumper-3_P1.3mm_Open_Pad1.0x1.5mm, B.Cu at (173.5, 91.9)
- added JP3: SolderJumper_3_Open, Jumper:SolderJumper-3_P1.3mm_Open_Pad1.0x1.5mm, B.Cu at (181.0, 69.2)
- added JP4: SolderJumper_3_Open, Jumper:SolderJumper-3_P1.3mm_Open_Pad1.0x1.5mm, B.Cu at (179.5, 72.8)
- added L1: DFE252012P-1R0M=P2, SamacSys_Parts:DFE2HCAH1R0MJ0L, F.Cu at (166.3, 89.2)
- added L2: DFE252012P-1R0M=P2, SamacSys_Parts:DFE2HCAH1R0MJ0L, F.Cu at (172.6, 70.8)
- added L3: DFE252012P-1R0M=P2, SamacSys_Parts:DFE2HCAH1R0MJ0L, F.Cu at (151.2, 79.5)
- added R1: 5k1, Resistor_SMD:R_0603_1608Metric, F.Cu at (203.9, 95.9)
- added R10: 20k, Resistor_SMD:R_0603_1608Metric, B.Cu at (180.1, 74.8)
- added R2: 5k1, Resistor_SMD:R_0603_1608Metric, F.Cu at (203.8, 98.9)
- added R3: 20k, Resistor_SMD:R_0603_1608Metric, B.Cu at (177.9, 89.2)
- added R4: 20k, Resistor_SMD:R_0603_1608Metric, B.Cu at (173.2, 93.9)
- added R5: 511k, Resistor_SMD:R_0603_1608Metric, F.Cu at (173.2, 87.5)
- added R6: 91k, Resistor_SMD:R_0603_1608Metric, F.Cu at (173.2, 89.0)
- added R7: 511k, Resistor_SMD:R_0603_1608Metric, F.Cu at (180.1, 69.0)
- added R8: 91k, Resistor_SMD:R_0603_1608Metric, F.Cu at (180.1, 70.5)
- added R9: 20k, Resistor_SMD:R_0603_1608Metric, B.Cu at (183.0, 70.1)
- added U2: TPS631000DRLR, SamacSys_Parts:SOTFL50P160X60-8N, F.Cu at (169.7, 88.0)
- added U3: TPS631000DRLR, SamacSys_Parts:SOTFL50P160X60-8N, F.Cu at (176.0, 69.6)
- added U4: BQ25622ERYKR, footprints:WQFN-HR18_RYK_TEX, F.Cu at (150.5, 83.4)
- moved IC1 136.7 mm to (217.8, 48.9)
Connections:
- IC1 pad 1: unconnected-(IC1-GND_1-Pad1) -> GND
- IC1 pad 13: unconnected-(IC1-IO19-Pad13) -> D-
- IC1 pad 14: unconnected-(IC1-IO20-Pad14) -> D+
- IC1 pad 2: unconnected-(IC1-3V3-Pad2) -> +3V3
- IC1 pad 40: unconnected-(IC1-GND_2-Pad40) -> GND
- IC1 pad 41: unconnected-(IC1-GND_3-Pad41) -> GND
- IC1 pad 42: unconnected-(IC1-GND_4-Pad42) -> GND
- IC1 pad 43: unconnected-(IC1-GND_5-Pad43) -> GND
- IC1 pad 44: unconnected-(IC1-GND_6-Pad44) -> GND
- IC1 pad 45: unconnected-(IC1-GND_7-Pad45) -> GND
- IC1 pad 46: unconnected-(IC1-GND_8-Pad46) -> GND
- IC1 pad 47: unconnected-(IC1-GND_9-Pad47) -> GND
- IC1 pad 48: unconnected-(IC1-GND_10-Pad48) -> GND
- IC1 pad 49: unconnected-(IC1-GND_11-Pad49) -> GND
- U1 pad P$72: unconnected-(U1-72-PadP$72) -> +5V
- U1 pad P$73: unconnected-(U1-73-PadP$73) -> GND
- U1 pad P$74: unconnected-(U1-74-PadP$74) -> +5V
- U1 pad P$75: unconnected-(U1-75-PadP$75) -> GND
Routing:
- net VDD: track 0.00 -> 11.7 mm
- net +5V: track 0.00 -> 8.48 mm, vias 0 -> 2
- net +3V3: track 0.00 -> 8.38 mm, vias 0 -> 2
- net 3V3_Mode: track 0.00 -> 7.52 mm, vias 0 -> 1
- net 3V3_En: track 0.00 -> 7.32 mm, vias 0 -> 1
- net 5V_En: track 0.00 -> 6.85 mm, vias 0 -> 1
- net GND: track 0.00 -> 6.70 mm, vias 0 -> 7
- net 5V_Mode: track 0.00 -> 6.43 mm, vias 0 -> 1
- net VBUS: track 0.00 -> 6.34 mm
- net SW: track 0.00 -> 5.05 mm, vias 0 -> 1
- net Net-(U3-LX1): track 0.00 -> 4.10 mm
- net FB5V: track 0.00 -> 3.96 mm
- net BTST: track 0.00 -> 3.81 mm, vias 0 -> 1
- net Net-(U2-LX1): track 0.00 -> 3.69 mm
- net FB3V3: track 0.00 -> 3.48 mm
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- added copper zone on B.Cu, net GND
- added copper zone on F.Cu, net GND
- removed copper zone on B.Cu, net (none)
- removed copper zone on F.Cu, net (none)
