File: ControlModule/CMBoard/CMBoard.kicad_sch (KiCad schematic)
At the start: 2 parts, among them IC1 ESP32-S3-WROOM-1U-N4

Commit message: Initial commit
Parts:
- removed 1: M.2-B-KEY-2280-ADAPTER, symbol M.2-Templates-eagle-import:M.2-B-KEY-2280-ADAPTER
- added U1: ~, M.2 Connectors:B+M 2280, symbol M.2 Connectors:B+M
Connections:
- net GND: now reaches IC1.1 (GND_1)
- net GND: now also IC1.40 (GND_2), IC1.41 (GND_3), IC1.42 (GND_4), IC1.43 (GND_5), IC1.44 (GND_6), IC1.45 (GND_7), IC1.46 (GND_8), IC1.47 (GND_9), IC1.48 (GND_10), IC1.49 (GND_11), U1.MP1, U1.P$73 (73), U1.P$75 (75)
- net D-: now reaches IC1.13 (IO19)
- net D+: now reaches IC1.14 (IO20)
- net +3V3: now reaches IC1.2 (3V3)
- new net +5V: U1.P$72 (72), U1.P$74 (74)
- no-connect marks 1 -> 0
Other:
- added sheet PSU (psu.kicad_sch)
- moved on the sheet: IC1
